File: ntc-6251-qmk-pcb.kicad_pcb (KiCad board)
At the start: 2 copper layers, 442 x 119 mm, 3 parts

Commit message: Finished schematic grid, connected footprints, prelim. arrangement of components on pcb
Parts:
- removed REF** (x2): 2U, Alps_Only:ALPS-2U
- removed REF**: 1U, Alps_Only:ALPS-1U
- added D1: D_Small, Diode_THT:D_DO-35_SOD27_P7.62mm_Horizontal, F.Cu at (52.6, 52.9)
- added D10: D_Small, Diode_THT:D_DO-35_SOD27_P7.62mm_Horizontal, F.Cu at (274.4, 135.5)
- added D100: D_Small, Diode_THT:D_DO-35_SOD27_P7.62mm_Horizontal, F.Cu at (243.8, 119.3)
- added D101: D_Small, Diode_THT:D_DO-35_SOD27_P7.62mm_Horizontal, F.Cu at (253.6, 136.5)
- added D102: D_Small, Diode_THT:D_DO-35_SOD27_P7.62mm_Horizontal, F.Cu at (397.5, 80.8)
- added D103: D_Small, Diode_THT:D_DO-35_SOD27_P7.62mm_Horizontal, F.Cu at (442.7, 99.3)
- added D11: D_Small, Diode_THT:D_DO-35_SOD27_P7.62mm_Horizontal, F.Cu at (357.5, 99.5)
- added D12: D_Small, Diode_THT:D_DO-35_SOD27_P7.62mm_Horizontal, F.Cu at (460.9, 99.8)
- added D13: D_Small, Diode_THT:D_DO-35_SOD27_P7.62mm_Horizontal, F.Cu at (73.2, 80.4)
- added D14: D_Small, Diode_THT:D_DO-35_SOD27_P7.62mm_Horizontal, F.Cu at (321.6, 80.0)
- added D15: D_Small, Diode_THT:D_DO-35_SOD27_P7.62mm_Horizontal, F.Cu at (288.8, 99.9)
- added D16: D_Small, Diode_THT:D_DO-35_SOD27_P7.62mm_Horizontal, F.Cu at (282.3, 119.3)
- added D17: D_Small, Diode_THT:D_DO-35_SOD27_P7.62mm_Horizontal, F.Cu at (307.6, 135.5)
- added D18: D_Small, Diode_THT:D_DO-35_SOD27_P7.62mm_Horizontal, F.Cu at (376.9, 99.8)
- added D19: D_Small, Diode_THT:D_DO-35_SOD27_P7.62mm_Horizontal, F.Cu at (480.0, 109.7)
- added D2: D_Small, Diode_THT:D_DO-35_SOD27_P7.62mm_Horizontal, F.Cu at (80.5, 52.9)
- added D20: D_Small, Diode_THT:D_DO-35_SOD27_P7.62mm_Horizontal, F.Cu at (92.7, 80.6)
- added D21: D_Small, Diode_THT:D_DO-35_SOD27_P7.62mm_Horizontal, F.Cu at (58.9, 99.7)
- added D22: D_Small, Diode_THT:D_DO-35_SOD27_P7.62mm_Horizontal, F.Cu at (318.0, 110.0)
- added D23: D_Small, Diode_THT:D_DO-35_SOD27_P7.62mm_Horizontal, F.Cu at (57.9, 136.0)
- added D24: D_Small, Diode_THT:D_DO-35_SOD27_P7.62mm_Horizontal, F.Cu at (60.8, 159.5)
- added D25: D_Small, Diode_THT:D_DO-35_SOD27_P7.62mm_Horizontal, F.Cu at (397.3, 100.7)
- added D26: D_Small, Diode_THT:D_DO-35_SOD27_P7.62mm_Horizontal, F.Cu at (422.6, 118.7)
- added D27: D_Small, Diode_THT:D_DO-35_SOD27_P7.62mm_Horizontal, F.Cu at (111.3, 80.3)
- added D28: D_Small, Diode_THT:D_DO-35_SOD27_P7.62mm_Horizontal, F.Cu at (80.5, 99.5)
- added D29: D_Small, Diode_THT:D_DO-35_SOD27_P7.62mm_Horizontal, F.Cu at (64.7, 119.3)
- added D3: D_Small, Diode_THT:D_DO-35_SOD27_P7.62mm_Horizontal, F.Cu at (100.0, 53.1)
- added D30: D_Small, Diode_THT:D_DO-35_SOD27_P7.62mm_Horizontal, F.Cu at (80.6, 136.1)
- added D31: D_Small, Diode_THT:D_DO-35_SOD27_P7.62mm_Horizontal, F.Cu at (97.2, 159.6)
- added D32: D_Small, Diode_THT:D_DO-35_SOD27_P7.62mm_Horizontal, F.Cu at (350.1, 158.3)
- added D33: D_Small, Diode_THT:D_DO-35_SOD27_P7.62mm_Horizontal, F.Cu at (443.8, 118.8)
- added D34: D_Small, Diode_THT:D_DO-35_SOD27_P7.62mm_Horizontal, F.Cu at (130.4, 80.5)
- added D35: D_Small, Diode_THT:D_DO-35_SOD27_P7.62mm_Horizontal, F.Cu at (100.0, 99.5)
- added D36: D_Small, Diode_THT:D_DO-35_SOD27_P7.62mm_Horizontal, F.Cu at (91.3, 119.4)
- added D37: D_Small, Diode_THT:D_DO-35_SOD27_P7.62mm_Horizontal, F.Cu at (100.3, 136.5)
- added D38: D_Small, Diode_THT:D_DO-35_SOD27_P7.62mm_Horizontal, F.Cu at (187.8, 158.4)
- added D39: D_Small, Diode_THT:D_DO-35_SOD27_P7.62mm_Horizontal, F.Cu at (369.9, 134.9)
- added D4: D_Small, Diode_THT:D_DO-35_SOD27_P7.62mm_Horizontal, F.Cu at (120.7, 53.6)
- added D40: D_Small, Diode_THT:D_DO-35_SOD27_P7.62mm_Horizontal, F.Cu at (462.7, 119.1)
- added D41: D_Small, Diode_THT:D_DO-35_SOD27_P7.62mm_Horizontal, F.Cu at (167.2, 53.9)
- added D42: D_Small, Diode_THT:D_DO-35_SOD27_P7.62mm_Horizontal, F.Cu at (149.6, 80.3)
- added D43: D_Small, Diode_THT:D_DO-35_SOD27_P7.62mm_Horizontal, F.Cu at (119.8, 99.4)
- added D44: D_Small, Diode_THT:D_DO-35_SOD27_P7.62mm_Horizontal, F.Cu at (111.0, 119.0)
- added D45: D_Small, Diode_THT:D_DO-35_SOD27_P7.62mm_Horizontal, F.Cu at (119.4, 136.6)
- added D46: D_Small, Diode_THT:D_DO-35_SOD27_P7.62mm_Horizontal, F.Cu at (273.5, 158.4)
- added D47: D_Small, Diode_THT:D_DO-35_SOD27_P7.62mm_Horizontal, F.Cu at (369.2, 158.2)
- added D48: D_Small, Diode_THT:D_DO-35_SOD27_P7.62mm_Horizontal, F.Cu at (423.4, 135.2)
- added D49: D_Small, Diode_THT:D_DO-35_SOD27_P7.62mm_Horizontal, F.Cu at (187.0, 54.1)
- added D5: D_Small, Diode_THT:D_DO-35_SOD27_P7.62mm_Horizontal, F.Cu at (140.9, 53.7)
- added D50: D_Small, Diode_THT:D_DO-35_SOD27_P7.62mm_Horizontal, F.Cu at (168.7, 79.8)
- added D51: D_Small, Diode_THT:D_DO-35_SOD27_P7.62mm_Horizontal, F.Cu at (139.0, 99.4)
- added D52: D_Small, Diode_THT:D_DO-35_SOD27_P7.62mm_Horizontal, F.Cu at (129.8, 119.0)
- added D53: D_Small, Diode_THT:D_DO-35_SOD27_P7.62mm_Horizontal, F.Cu at (139.1, 136.2)
- added D54: D_Small, Diode_THT:D_DO-35_SOD27_P7.62mm_Horizontal, F.Cu at (321.1, 158.2)
- added D55: D_Small, Diode_THT:D_DO-35_SOD27_P7.62mm_Horizontal, F.Cu at (388.8, 158.3)
- added D56: D_Small, Diode_THT:D_DO-35_SOD27_P7.62mm_Horizontal, F.Cu at (444.2, 136.8)
- added D57: D_Small, Diode_THT:D_DO-35_SOD27_P7.62mm_Horizontal, F.Cu at (205.5, 54.4)
- added D58: D_Small, Diode_THT:D_DO-35_SOD27_P7.62mm_Horizontal, F.Cu at (187.1, 80.3)
- added D59: D_Small, Diode_THT:D_DO-35_SOD27_P7.62mm_Horizontal, F.Cu at (157.9, 99.2)
- added D6: D_Small, Diode_THT:D_DO-35_SOD27_P7.62mm_Horizontal, F.Cu at (53.4, 80.5)
- added D60: D_Small, Diode_THT:D_DO-35_SOD27_P7.62mm_Horizontal, F.Cu at (147.8, 118.8)
- added D61: D_Small, Diode_THT:D_DO-35_SOD27_P7.62mm_Horizontal, F.Cu at (158.8, 135.8)
- added D62: D_Small, Diode_THT:D_DO-35_SOD27_P7.62mm_Horizontal, F.Cu at (357.6, 53.4)
- added D63: D_Small, Diode_THT:D_DO-35_SOD27_P7.62mm_Horizontal, F.Cu at (422.0, 79.9)
- added D64: D_Small, Diode_THT:D_DO-35_SOD27_P7.62mm_Horizontal, F.Cu at (462.9, 136.2)
- added D65: D_Small, Diode_THT:D_DO-35_SOD27_P7.62mm_Horizontal, F.Cu at (224.6, 54.1)
- added D66: D_Small, Diode_THT:D_DO-35_SOD27_P7.62mm_Horizontal, F.Cu at (206.0, 80.4)
- added D67: D_Small, Diode_THT:D_DO-35_SOD27_P7.62mm_Horizontal, F.Cu at (177.4, 99.2)
- added D68: D_Small, Diode_THT:D_DO-35_SOD27_P7.62mm_Horizontal, F.Cu at (166.7, 118.7)
- added D69: D_Small, Diode_THT:D_DO-35_SOD27_P7.62mm_Horizontal, F.Cu at (177.6, 136.2)
- added D7: D_Small, Diode_THT:D_DO-35_SOD27_P7.62mm_Horizontal, F.Cu at (301.7, 80.2)
- added D70: D_Small, Diode_THT:D_DO-35_SOD27_P7.62mm_Horizontal, F.Cu at (377.4, 53.5)
- added D71: D_Small, Diode_THT:D_DO-35_SOD27_P7.62mm_Horizontal, F.Cu at (440.7, 80.8)
- added D72: D_Small, Diode_THT:D_DO-35_SOD27_P7.62mm_Horizontal, F.Cu at (480.8, 146.5)
- added D73: D_Small, Diode_THT:D_DO-35_SOD27_P7.62mm_Horizontal, F.Cu at (248.9, 54.1)
- added D74: D_Small, Diode_THT:D_DO-35_SOD27_P7.62mm_Horizontal, F.Cu at (225.4, 80.8)
- added D75: D_Small, Diode_THT:D_DO-35_SOD27_P7.62mm_Horizontal, F.Cu at (196.3, 100.0)
- added D76: D_Small, Diode_THT:D_DO-35_SOD27_P7.62mm_Horizontal, F.Cu at (185.7, 118.9)
- added D77: D_Small, Diode_THT:D_DO-35_SOD27_P7.62mm_Horizontal, F.Cu at (196.5, 135.5)
- added D78: D_Small, Diode_THT:D_DO-35_SOD27_P7.62mm_Horizontal, F.Cu at (396.1, 53.3)
- added D79: D_Small, Diode_THT:D_DO-35_SOD27_P7.62mm_Horizontal, F.Cu at (459.6, 79.6)
- added D8: D_Small, Diode_THT:D_DO-35_SOD27_P7.62mm_Horizontal, F.Cu at (272.3, 100.2)
- added D80: D_Small, Diode_THT:D_DO-35_SOD27_P7.62mm_Horizontal, F.Cu at (429.2, 158.6)
- added D81: D_Small, Diode_THT:D_DO-35_SOD27_P7.62mm_Horizontal, F.Cu at (268.8, 54.1)
- added D82: D_Small, Diode_THT:D_DO-35_SOD27_P7.62mm_Horizontal, F.Cu at (244.8, 80.8)
- added D83: D_Small, Diode_THT:D_DO-35_SOD27_P7.62mm_Horizontal, F.Cu at (215.9, 100.1)
- added D84: D_Small, Diode_THT:D_DO-35_SOD27_P7.62mm_Horizontal, F.Cu at (205.0, 119.2)
- added D85: D_Small, Diode_THT:D_DO-35_SOD27_P7.62mm_Horizontal, F.Cu at (215.9, 136.0)
- added D86: D_Small, Diode_THT:D_DO-35_SOD27_P7.62mm_Horizontal, F.Cu at (357.6, 80.0)
- added D87: D_Small, Diode_THT:D_DO-35_SOD27_P7.62mm_Horizontal, F.Cu at (478.0, 80.1)
- added D88: D_Small, Diode_THT:D_DO-35_SOD27_P7.62mm_Horizontal, F.Cu at (461.8, 158.9)
- added D89: D_Small, Diode_THT:D_DO-35_SOD27_P7.62mm_Horizontal, F.Cu at (288.1, 54.0)
- added D9: D_Small, Diode_THT:D_DO-35_SOD27_P7.62mm_Horizontal, F.Cu at (262.4, 119.2)
- added D90: D_Small, Diode_THT:D_DO-35_SOD27_P7.62mm_Horizontal, F.Cu at (263.4, 80.1)
- added D91: D_Small, Diode_THT:D_DO-35_SOD27_P7.62mm_Horizontal, F.Cu at (234.7, 100.0)
- added D92: D_Small, Diode_THT:D_DO-35_SOD27_P7.62mm_Horizontal, F.Cu at (224.5, 119.5)
- added D93: D_Small, Diode_THT:D_DO-35_SOD27_P7.62mm_Horizontal, F.Cu at (234.8, 136.2)
- added D94: D_Small, Diode_THT:D_DO-35_SOD27_P7.62mm_Horizontal, F.Cu at (377.4, 79.5)
- added D95: D_Small, Diode_THT:D_DO-35_SOD27_P7.62mm_Horizontal, F.Cu at (421.9, 99.6)
- added D97: D_Small, Diode_THT:D_DO-35_SOD27_P7.62mm_Horizontal, F.Cu at (307.4, 54.1)
- added D98: D_Small, Diode_THT:D_DO-35_SOD27_P7.62mm_Horizontal, F.Cu at (282.4, 79.8)
- added D99: D_Small, Diode_THT:D_DO-35_SOD27_P7.62mm_Horizontal, F.Cu at (253.8, 99.8)
- added MX1: MX-NoLED, Alps_Only:ALPS-1U, F.Cu at (42.0, 49.7)
- added MX10: MX-NoLED, Alps_Only:ALPS-1U, F.Cu at (264.6, 132.2)
- added MX100: MX-NoLED, Alps_Only:ALPS-1U, F.Cu at (234.7, 115.6)
- added MX101: MX-NoLED, Alps_Only:ALPS-1U, F.Cu at (244.8, 132.2)
- added MX102: MX-NoLED, Alps_Only:ALPS-1U, F.Cu at (387.6, 76.6)
- added MX103: MX-NoLED, Alps_Only:ALPS-1U, F.Cu at (433.6, 96.2)
- added MX11: MX-NoLED, Alps_Only:ALPS-1U, F.Cu at (348.7, 96.2)
- added MX12: MX-NoLED, Alps_Only:ALPS-1U, F.Cu at (452.4, 96.2)
- added MX13: MX-NoLED, Alps_Only:ALPS-1U, F.Cu at (63.0, 76.6)
- added MX14: MX-NoLED, Alps_Only:ALPS-1U, F.Cu at (311.5, 76.6)
- added MX15: MX-NoLED, Alps_Only:ALPS-1U, F.Cu at (282.0, 96.2)
- added MX16: MX-NoLED, Alps_Only:ALPS-1U, F.Cu at (273.4, 115.6)
- added MX17: MX-NoLED, Alps_Only:ALPS-1U, F.Cu at (299.8, 132.2)
- added MX18: MX-NoLED, Alps_Only:ALPS-1U, F.Cu at (366.6, 96.2)
- added MX19: MX-NoLED, Alps_Only:ALPS-1U, F.Cu at (472.4, 105.9)
- added MX2: MX-NoLED, Alps_Only:ALPS-1U, F.Cu at (70.8, 49.7)
- added MX20: MX-NoLED, Alps_Only:ALPS-1U, F.Cu at (83.0, 76.6)
- added MX21: MX-NoLED, Alps_Only:ALPS-1U, F.Cu at (49.7, 96.2)
- added MX22: MX-NoLED, Alps_Only:ALPS-1U, F.Cu at (308.0, 106.6)
- added MX23: MX-NoLED, Alps_Only:ALPS-1U, F.Cu at (48.3, 132.2)
- added MX24: MX-NoLED, Alps_Only:ALPS-1U, F.Cu at (51.0, 155.4)
- added MX25: MX-NoLED, Alps_Only:ALPS-1U, F.Cu at (387.2, 96.2)
- added MX26: MX-NoLED, Alps_Only:ALPS-1U, F.Cu at (413.4, 115.6)
- added MX27: MX-NoLED, Alps_Only:ALPS-1U, F.Cu at (102.0, 76.6)
- added MX28: MX-NoLED, Alps_Only:ALPS-1U, F.Cu at (71.1, 96.2)
- added MX29: MX-NoLED, Alps_Only:ALPS-1U, F.Cu at (55.4, 115.6)
- added MX3: MX-NoLED, Alps_Only:ALPS-1U, F.Cu at (90.2, 49.7)
- added MX30: MX-NoLED, Alps_Only:ALPS-1U, F.Cu at (71.0, 132.2)
- added MX31: MX-NoLED, Alps_Only:ALPS-1U, F.Cu at (87.5, 155.4)
- added MX32: MX-NoLED, Alps_Only:ALPS-1U, F.Cu at (342.6, 155.4)
- added MX33: MX-NoLED, Alps_Only:ALPS-1U, F.Cu at (434.2, 115.6)
- added MX34: MX-NoLED, Alps_Only:ALPS-1U, F.Cu at (121.0, 76.6)
- added MX35: MX-NoLED, Alps_Only:ALPS-1U, F.Cu at (90.7, 96.2)
- added MX36: MX-NoLED, Alps_Only:ALPS-1U, F.Cu at (82.5, 115.6)
- added MX37: MX-NoLED, Alps_Only:ALPS-1U, F.Cu at (90.5, 132.2)
- added MX38: MX-NoLED, Alps_Only:ALPS-1U, F.Cu at (178.1, 155.4)
- added MX39: MX-NoLED, Alps_Only:ALPS-1U, F.Cu at (362.0, 132.2)
- added MX4: MX-NoLED, Alps_Only:ALPS-1U, F.Cu at (110.7, 49.7)
- added MX40: MX-NoLED, Alps_Only:ALPS-1U, F.Cu at (454.0, 115.6)
- added MX41: MX-NoLED, Alps_Only:ALPS-1U, F.Cu at (157.8, 49.7)
- added MX42: MX-NoLED, Alps_Only:ALPS-1U, F.Cu at (140.1, 76.6)
- added MX43: MX-NoLED, Alps_Only:ALPS-1U, F.Cu at (110.5, 96.2)
- added MX44: MX-NoLED, Alps_Only:ALPS-1U, F.Cu at (101.9, 115.6)
- added MX45: MX-NoLED, Alps_Only:ALPS-1U, F.Cu at (110.1, 132.2)
- added MX46: MX-NoLED, Alps_Only:ALPS-1U, F.Cu at (264.4, 155.4)
- added MX47: MX-NoLED, Alps_Only:ALPS-1U, F.Cu at (361.2, 155.4)
- added MX48: MX-NoLED, Alps_Only:ALPS-1U, F.Cu at (413.9, 132.2)
- added MX49: MX-NoLED, Alps_Only:ALPS-1U, F.Cu at (177.5, 49.7)
- added MX5: MX-NoLED, Alps_Only:ALPS-1U, F.Cu at (130.3, 49.7)
- added MX50: MX-NoLED, Alps_Only:ALPS-1U, F.Cu at (159.1, 76.6)
- added MX51: MX-NoLED, Alps_Only:ALPS-1U, F.Cu at (129.2, 96.2)
- added MX52: MX-NoLED, Alps_Only:ALPS-1U, F.Cu at (120.8, 115.6)
- added MX53: MX-NoLED, Alps_Only:ALPS-1U, F.Cu at (129.2, 132.2)
- added MX54: MX-NoLED, Alps_Only:ALPS-1U, F.Cu at (311.0, 155.4)
- added MX55: MX-NoLED, Alps_Only:ALPS-1U, F.Cu at (382.5, 155.4)
- added MX56: MX-NoLED, Alps_Only:ALPS-1U, F.Cu at (434.7, 132.2)
- added MX57: MX-NoLED, Alps_Only:ALPS-1U, F.Cu at (196.7, 49.7)
- added MX58: MX-NoLED, Alps_Only:ALPS-1U, F.Cu at (177.9, 76.6)
- added MX59: MX-NoLED, Alps_Only:ALPS-1U, F.Cu at (148.3, 96.2)
- added MX6: MX-NoLED, Alps_Only:ALPS-1U, F.Cu at (44.2, 76.6)
- added MX60: MX-NoLED, Alps_Only:ALPS-1U, F.Cu at (138.6, 115.6)
- added MX61: MX-NoLED, Alps_Only:ALPS-1U, F.Cu at (149.1, 132.2)
- added MX62: MX-NoLED, Alps_Only:ALPS-1U, F.Cu at (348.2, 49.7)
- added MX63: MX-NoLED, Alps_Only:ALPS-1U, F.Cu at (413.6, 76.6)
- added MX64: MX-NoLED, Alps_Only:ALPS-1U, F.Cu at (453.7, 132.2)
- added MX65: MX-NoLED, Alps_Only:ALPS-1U, F.Cu at (215.1, 49.7)
- added MX66: MX-NoLED, Alps_Only:ALPS-1U, F.Cu at (196.8, 76.6)
- added MX67: MX-NoLED, Alps_Only:ALPS-1U, F.Cu at (167.7, 96.2)
- added MX68: MX-NoLED, Alps_Only:ALPS-1U, F.Cu at (157.9, 115.6)
- added MX69: MX-NoLED, Alps_Only:ALPS-1U, F.Cu at (168.2, 132.2)
- added MX7: MX-NoLED, Alps_Only:ALPS-1U, F.Cu at (292.4, 76.6)
- added MX70: MX-NoLED, Alps_Only:ALPS-1U, F.Cu at (367.6, 49.7)
- added MX71: MX-NoLED, Alps_Only:ALPS-1U, F.Cu at (431.3, 76.6)
- added MX72: MX-NoLED, Alps_Only:ALPS-1U, F.Cu at (473.8, 143.8)
- added MX73: MX-NoLED, Alps_Only:ALPS-1U, F.Cu at (239.4, 49.7)
- added MX74: MX-NoLED, Alps_Only:ALPS-1U, F.Cu at (216.2, 76.6)
- added MX75: MX-NoLED, Alps_Only:ALPS-1U, F.Cu at (187.1, 96.2)
- added MX76: MX-NoLED, Alps_Only:ALPS-1U, F.Cu at (176.6, 115.6)
- added MX77: MX-NoLED, Alps_Only:ALPS-1U, F.Cu at (186.9, 132.2)
- added MX78: MX-NoLED, Alps_Only:ALPS-1U, F.Cu at (386.8, 49.7)
- added MX79: MX-NoLED, Alps_Only:ALPS-1U, F.Cu at (450.1, 76.6)
- added MX8: MX-NoLED, Alps_Only:ALPS-1U, F.Cu at (263.1, 96.2)
- added MX80: MX-NoLED, Alps_Only:ALPS-1U, F.Cu at (418.4, 155.4)
- added MX81: MX-NoLED, Alps_Only:ALPS-1U, F.Cu at (259.3, 49.7)
- added MX82: MX-NoLED, Alps_Only:ALPS-1U, F.Cu at (235.5, 76.6)
- added MX83: MX-NoLED, Alps_Only:ALPS-1U, F.Cu at (206.0, 96.2)
- added MX84: MX-NoLED, Alps_Only:ALPS-1U, F.Cu at (196.0, 115.6)
- added MX85: MX-NoLED, Alps_Only:ALPS-1U, F.Cu at (206.2, 132.2)
- added MX86: MX-NoLED, Alps_Only:ALPS-1U, F.Cu at (348.1, 76.6)
- added MX87: MX-NoLED, Alps_Only:ALPS-1U, F.Cu at (469.5, 76.6)
- added MX88: MX-NoLED, Alps_Only:ALPS-1U, F.Cu at (451.9, 155.4)
- added MX89: MX-NoLED, Alps_Only:ALPS-1U, F.Cu at (278.4, 49.7)
- added MX9: MX-NoLED, Alps_Only:ALPS-1U, F.Cu at (253.5, 115.6)
- added MX90: MX-NoLED, Alps_Only:ALPS-1U, F.Cu at (254.3, 76.6)
- added MX91: MX-NoLED, Alps_Only:ALPS-1U, F.Cu at (225.1, 96.2)
- added MX92: MX-NoLED, Alps_Only:ALPS-1U, F.Cu at (214.9, 115.6)
- added MX93: MX-NoLED, Alps_Only:ALPS-1U, F.Cu at (225.6, 132.2)
- added MX94: MX-NoLED, Alps_Only:ALPS-1U, F.Cu at (368.1, 76.6)
- added MX95: MX-NoLED, Alps_Only:ALPS-1U, F.Cu at (413.3, 96.2)
- added MX97: MX-NoLED, Alps_Only:ALPS-1U, F.Cu at (297.3, 49.7)
- added MX98: MX-NoLED, Alps_Only:ALPS-1U, F.Cu at (273.2, 76.6)
- added MX99: MX-NoLED, Alps_Only:ALPS-1U, F.Cu at (244.5, 96.2)
- added U1: ATMEGA32U4, Package_QFP:TQFP-44_10x10mm_P0.8mm, F.Cu at (416.6, 51.2)

Commit message: Updates
Parts:
- moved D48 48.3 mm to (420.6, 183.4)
- moved D56 44.0 mm to (441.9, 180.7)
- moved D62 32.0 mm to (389.5, 49.9)
- moved D79 25.8 mm to (485.3, 81.5)
- moved D70 25.8 mm to (396.3, 35.9)
- moved D40 24.0 mm to (486.4, 122.6)
- moved D80 20.6 mm to (427.6, 179.2)
- moved D12 20.2 mm to (481.1, 97.8)
- moved D88 20.0 mm to (475.6, 173.3)
- moved MX22 19.2 mm to (296.1, 121.7)
- moved D64 16.0 mm to (478.8, 135.4)
- moved MX56 14.3 mm to (423.2, 140.8)
- moved MX64 14.3 mm to (442.2, 140.8)
- moved MX102 14.2 mm to (375.3, 83.6)
- moved MX72 14.1 mm to (461.3, 150.4), turned to 90 degrees
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Other:
- board size 442 x 119 mm -> 432 x 109.1 mm

Commit message: Finished aligning switches and diodes
Parts:
- moved U1 78.1 mm to (378.1, 121.8), turned to 270 degrees
- moved D62 64.0 mm to (327.7, 66.5)
- moved D70 58.2 mm to (346.7, 66.5)
- moved D48 40.1 mm to (413.7, 143.9)
- moved D56 38.0 mm to (432.7, 143.9)
- moved D40 34.7 mm to (451.8, 124.8)
- moved D79 34.0 mm to (451.8, 86.8)
- moved D78 33.0 mm to (365.8, 66.5)
- moved D12 30.4 mm to (451.8, 105.8)
- moved D64 28.4 mm to (451.8, 143.9)
- moved D88 27.6 mm to (451.8, 159.6)
- moved D87 25.5 mm to (456.1, 93.2), turned to 0 degrees
- moved D72 24.9 mm to (464.4, 140.8), turned to 180 degrees
- moved D80 20.1 mm to (423.0, 159.6)
- moved D22 19.2 mm to (305.7, 124.8)
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