File: ntc-6251-qmk-pcb.kicad_pcb (KiCad board)
At the start: 2 copper layers, 432 x 109.1 mm, 208 parts

Commit message: Updated layout
Parts:
- removed REF**: WeAct BlackPill, STM32:YAAJ_WeAct_BlackPill_SWD_2
- added J1: USB_B, Connector_USB:USB_B_OST_USB-B1HSxx_Horizontal, B.Cu at (393.1, 61.9)
- added R1: R_Small, Resistor_THT:R_Axial_DIN0207_L6.3mm_D2.5mm_P7.62mm_Horizontal, F.Cu at (401.9, 67.8)
- added R2: R_Small, Resistor_THT:R_Axial_DIN0207_L6.3mm_D2.5mm_P7.62mm_Horizontal, F.Cu at (425.1, 67.8)
- added R3: R_Small, Resistor_THT:R_Axial_DIN0207_L6.3mm_D2.5mm_P7.62mm_Horizontal, F.Cu at (448.3, 67.8)
- added U1: YAAJ_WeAct_BlackPill_Part_Like_SWD_Breakout, STM32:YAAJ_WeAct_BlackPill_SWD_2, F.Cu at (366.9, 114.1)
- turned D1 to 180 degrees
Connections:
- D104 pad 2: Net-(D104-Pad2) -> +3V3
- D105 pad 2: Net-(D105-Pad2) -> +3V3
- D96 pad 2: Net-(D96-Pad2) -> +3V3
- MX1 pad 1: Col3 -> Col1
- MX102 pad 1: Col3 -> Col1
- MX11 pad 1: Col1 -> Col3
- MX20 pad 1: Col1 -> Col3
- MX21 pad 1: Col3 -> Col1
- MX23 pad 1: Col3 -> Col1
- MX24 pad 1: Col3 -> Col1
- MX25 pad 1: Col3 -> Col1
- MX29 pad 1: Col3 -> Col1
- MX3 pad 1: Col1 -> Col3
- MX31 pad 1: Col1 -> Col3
- MX32 pad 1: Col2 -> Col6
- MX35 pad 1: Col1 -> Col3
- MX37 pad 1: Col1 -> Col3
- MX39 pad 1: Col6 -> Col7
- MX44 pad 1: Col1 -> Col3
- MX47 pad 1: Col4 -> Col5
- MX55 pad 1: Col5 -> Col4
- MX6 pad 1: Col3 -> Col1
- MX62 pad 1: Net-(MX62-Pad1) -> Col6
- MX70 pad 1: Col6 -> Col5
- MX78 pad 1: Col5 -> Col4
- MX86 pad 1: Col1 -> Col3
Routing:
- net Col6: track 0.00 -> 652.1 mm, vias 0 -> 1
- net Col5: track 0.00 -> 638.2 mm, vias 0 -> 1
- net Col4: track 0.00 -> 635.6 mm, vias 0 -> 1
- net Col7: track 0.00 -> 634.2 mm, vias 0 -> 2
- net Col8: track 0.00 -> 579.7 mm, vias 0 -> 3
- net Col1: track 0.00 -> 520.0 mm
- net Col13: track 0.00 -> 495.2 mm, vias 0 -> 1
- net Col2: track 0.00 -> 475.8 mm, vias 0 -> 1
- net Col3: track 0.00 -> 464.4 mm, vias 0 -> 1
- net Row6: track 0.00 -> 462.5 mm
- net Col10: track 0.00 -> 454.5 mm, vias 0 -> 1
- net Col11: track 0.00 -> 450.8 mm, vias 0 -> 2
- net Col12: track 0.00 -> 445.8 mm, vias 0 -> 1
- net Col9: track 0.00 -> 413.5 mm, vias 0 -> 1
- net Row1: track 0.00 -> 354.6 mm
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
Commit message: Finished most of small issues with traces
Parts:
- added G***: HVAJ, keyboard_parts:vicky_logo, F.Cu at (332.4, 140.6)
Routing:
- net Row6: track 462.5 -> 480.9 mm
- net Row8: track 263.8 -> 276.6 mm
- net Col8: track 579.7 -> 569.7 mm
- net Net-(D99-Pad2): track 0.00 -> 7.03 mm
- net Col12: track 445.8 -> 450.4 mm
- net Row1: track 354.6 -> 350.2 mm
- net Col3: track 464.4 -> 460.5 mm
- net Col2: track 475.8 -> 471.9 mm
- net Col5: track 638.2 -> 634.4 mm
- net Col4: track 635.6 -> 632.0 mm
- net Col6: track 652.1 -> 654.9 mm
- net Col10: track 454.5 -> 457.2 mm
- net Col7: track 634.2 -> 631.9 mm
- net Row7: track 287.3 -> 289.4 mm
- net Row5: track 304.0 -> 305.5 mm
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
Commit message: Changed connector fixed controller pins, re-routed all traces near controller
Parts:
- removed G***: HVAJ, keyboard_parts:vicky_logo
- J1: value USB_B -> Conn_01x04_Male; footprint Connector_USB:USB_B_OST_USB-B1HSxx_Horizontal -> Connector_PinHeader_2.54mm:PinHeader_1x04_P2.54mm_Horizontal; moved to F.Cu
- moved J1 4.83 mm to (389.8, 58.4)
- moved U1 2.90 mm to (369.9, 114.1)
Connections:
- J1 pad 1: +5V -> GND
- J1 pad 2: D- -> D+
- J1 pad 3: D+ -> D-
- J1 pad 4: GND -> +5V
- U1 pad 18: Col7 -> Net-(U1-Pad18)
- U1 pad 19: Col8 -> Net-(U1-Pad19)
- U1 pad 20: Col9 -> Net-(U1-Pad20)
- U1 pad 21: Col10 -> Col7
- U1 pad 22: Col11 -> Col8
- U1 pad 23: Col12 -> Col9
- U1 pad 24: Col13 -> Col10
- U1 pad 25: Net-(U1-Pad25) -> Col11
- U1 pad 26: Net-(U1-Pad26) -> Col12
- U1 pad 27: Net-(U1-Pad27) -> Col13
Routing:
- net Row7: track 289.4 -> 409.7 mm
- net Col6: track 654.9 -> 588.9 mm, vias 1 -> 2
- net Col7: track 631.9 -> 569.8 mm
- net Col12: track 450.4 -> 508.8 mm, vias 1 -> 0
- net Col8: track 569.7 -> 624.8 mm, vias 3 -> 2
- net Col5: track 634.4 -> 589.8 mm, vias 1 -> 2
- net Col4: track 632.0 -> 597.1 mm, vias 1 -> 2
- net Row8: track 276.6 -> 300.9 mm
- net Col9: track 413.7 -> 435.2 mm
- net GND: track 101.2 -> 84.1 mm
- net Row1: track 350.2 -> 363.7 mm
- net Col10: track 457.2 -> 445.1 mm
- net Net-(J1-Pad5): track 12.0 -> 0.00 mm
- net Row2: track 324.8 -> 335.1 mm
- net Row4: track 299.0 -> 309.1 mm
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
Commit message: Last fixes and copper pour on rounded pcb
Routing:
- net Row7: track 409.7 -> 409.1 mm

Commit message: Last small fixes before printing
Parts:
- added G***: HVAJ, ntc-pcb:vicky_logo, F.Cu at (379.3, 140.8)
Routing:
- net Col7: track 569.8 -> 581.5 mm
- net Col8: track 624.8 -> 636.3 mm
- net Row3: track 319.1 -> 324.7 mm
- net Row2: track 335.1 -> 338.2 mm
- net Row6: track 478.7 -> 475.9 mm
- net Col12: track 508.8 -> 510.8 mm
- added copper zone on B.Cu, net (none)
- added copper zone on F.Cu, net (none)
