File: ntc-6251-qmk-pcb.sch (KiCad schematic (older format))
At the start: 237 parts, among them J1 Conn_01x04, J2 Conn_01x04, U1 ATmega32A-PU

Commit message: Finished schematic grid, connected footprints, prelim. arrangement of components on pcb
Parts:
- removed AVR1: AVR-ISP-6, Connector_PinHeader_2.54mm:PinHeader_2x03_P2.54mm_Horizontal, symbol Connector:AVR-ISP-6
- removed Boot1: Boot, Button_Switch_THT:SW_PUSH_6mm, symbol Switch:SW_Push
- removed C1: 4.7u, Capacitor_THT:CP_Radial_D5.0mm_P2.50mm, symbol Device:CP1
- removed C2, C3: 0.1u, Capacitor_THT:C_Disc_D3.0mm_W2.0mm_P2.50mm, symbol Device:C
- removed C4, C5: 22p, Capacitor_THT:C_Disc_D6.0mm_W2.5mm_P5.00mm, symbol Device:C_Small
- removed D1, D2: 3.6V, Diode_THT:D_DO-35_SOD27_P7.62mm_Horizontal, symbol Device:D_Zener
- removed D104, D105, D106, D107, D96: D_Small, custom_parts:D_DO-35_SOD27_P7.62mm_Horizontal, symbol Device:D_Small
- removed F1: 500mA, Fuse:Fuse_Littelfuse_395Series, symbol Device:Polyfuse
- removed H1, H2: MountingHole_Pad, custom_parts:screw-hole, symbol Mechanical:MountingHole_Pad
- removed J1, J2: Conn_01x04, Connector_JST:JST_PH_S4B-PH-K_1x04_P2.00mm_Horizontal, symbol Connector_Generic:Conn_01x04
- removed LED1, LED2, LED3: LED, LED_THT:LED_D5.0mm, symbol Device:LED
- removed MX104, MX105, MX96: MX-NoLED, Alps_Only:ALPS-1U, symbol MX_Alps_Hybrid:MX-NoLED
- removed R1, R5, R6, R7: 1.5K, Resistor_THT:R_Axial_DIN0207_L6.3mm_D2.5mm_P10.16mm_Horizontal, symbol Device:R
- removed R2, R3: 68R, Resistor_THT:R_Axial_DIN0207_L6.3mm_D2.5mm_P10.16mm_Horizontal, symbol Device:R
- removed R4: 10k, Resistor_THT:R_Axial_DIN0207_L6.3mm_D2.5mm_P10.16mm_Horizontal, symbol Device:R
- removed Reset1: Reset, Button_Switch_THT:SW_PUSH_6mm, symbol Switch:SW_Push
- removed U1: ATmega32A-PU, Package_DIP:DIP-40_W15.24mm_Socket, symbol MCU_Microchip_ATmega:ATmega32A-PU
- removed XTAL1: Crystal, Crystal:Crystal_HC49-4H_Vertical, symbol Device:Crystal
- added D1, D2: D_Small, Diode_THT:D_DO-35_SOD27_P7.62mm_Horizontal, symbol Device:D_Small
- added U1: ATMEGA32U4, Package_QFP:TQFP-44_10x10mm_P0.8mm, symbol keyboard_parts:ATMEGA32U4
- D10, D100, D101, D102, D103, D11, D12, D13, D14, D15, D16, D17, D18, D19, D20, D21, D22, D23, D24, D25, D26, D27, D28, D29, D3, D30, D31, D32, D33, D34, D35, D36, D37, D38, D39, D4, D40, D41, D42, D43, D44, D45, D46, D47, D48, D49, D5, D50, D51, D52, D53, D54, D55, D56, D57, D58, D59, D6, D60, D61, D62, D63, D64, D65, D66, D67, D68, D69, D7, D70, D71, D72, D73, D74, D75, D76, D77, D78, D79, D8, D80, D81, D82, D83, D84, D85, D86, D87, D88, D89, D9, D90, D91, D92, D93, D94, D95, D97, D98, D99: footprint custom_parts:D_DO-35_SOD27_P7.62mm_Horizontal -> Diode_THT:D_DO-35_SOD27_P7.62mm_Horizontal
- MX100, MX102, MX26: footprint Alps_Only:ALPS-2U -> Alps_Only:ALPS-1U
- MX27, MX40, MX67, MX69, MX75, MX77: footprint Alps_Only:ALPS-1.5U -> Alps_Only:ALPS-1U
- MX41: footprint Alps_Only:ALPS-1.75U -> Alps_Only:ALPS-1U
- MX54, MX55: footprint Alps_Only:ALPS-2.25U -> Alps_Only:ALPS-1U
- MX66: footprint Alps_Only:ALPS-2.75U -> Alps_Only:ALPS-1U
- MX68, MX76: footprint Alps_Only:ALPS-1.25U -> Alps_Only:ALPS-1U
Connections:
- net labels added: Col1, Col10, Col11, Col12, Col13, Col2, Col3, Col4, Col5, Col6, Col7, Col8, Col9, Row1, Row2, Row3, Row4, Row5, Row6, Row7, Row8
- net labels removed: +5V, D+, D-, GND, JST-D+, JST-D-, MISO, MOSI, SCK, VCC, boot, caps, col0, col1, col10, col11, col12, col13, col2, col3, col4, col5, col6, col7, col8, col9, num, reset, row0, row1, row2, row3, row4, row5, row6, row7, scroll
- wire segments 344 -> 306

Commit message: Updates
Parts:
- added C? (x2): 22p, symbol Device:C_Small
- added C? (x5): 0.1u, symbol Device:C_Small
- added C?: 1u, symbol Device:C_Small
- added R?: 10k, symbol Device:R_Small
- added Y?: XTAL, symbol Device:Crystal_GND24
Connections:
- net labels added: +5V, GND, XTAL1, XTAL2
- wire segments 306 -> 346

Commit message: Better matrix layout
Parts:
- removed C? (x2): 22p, symbol Device:C_Small
- removed C? (x5): 0.1u, symbol Device:C_Small
- removed C?: 1u, symbol Device:C_Small
- removed R?: 10k, symbol Device:R_Small
- removed Y?: XTAL, symbol Device:Crystal_GND24
- U1: footprint Package_QFP:TQFP-44_10x10mm_P0.8mm -> (none)
Connections:
- wire segments 346 -> 307
Other:
- moved on the sheet: D1, D10, D100, D101, D102, D103, D11, D12, D14, D15, D16, D17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

Commit message: Updated layout
Parts:
- removed U1: ATMEGA32U4, symbol keyboard_parts:ATMEGA32U4
- added D104, D105, D96: LED, LED_THT:LED_Rectangular_W5.0mm_H2.0mm, symbol Device:LED
- added J1: USB_B, Connector_USB:USB_B_OST_USB-B1HSxx_Horizontal, symbol Connector:USB_B
- added R1, R2, R3: R_Small, Resistor_THT:R_Axial_DIN0207_L6.3mm_D2.5mm_P7.62mm_Horizontal, symbol Device:R_Small
- added U1: YAAJ_WeAct_BlackPill_Part_Like_SWD_Breakout, STM32:YAAJ_WeAct_BlackPill_SWD_2, symbol YAAJ_WeAct_BlackPill_Part_Like_SWD_Breakout:YAAJ_WeAct_BlackPill_Part_Like_SWD_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
Connections:
- net +5V: now also J1.1 (VBUS), U1.40 (5V)
- net Col1: now also MX1.1 (COL), MX102.1 (COL), MX21.1 (COL), MX23.1 (COL), MX24.1 (COL), MX25.1 (COL), MX29.1 (COL), MX6.1 (COL), U1.12 (PB4); no longer MX11.1 (COL), MX20.1 (COL), MX3.1 (COL), MX31.1 (COL), MX35.1 (COL), MX37.1 (COL), MX44.1 (COL), MX86.1 (COL)
- net Col10: now also U1.21 (VBat)
- net Col11: now also U1.22 (PC13)
- net Col12: now also U1.23 (PC14)
- net Col13: now also U1.24 (PC15)
- net Col2: now also U1.13 (PB5); no longer MX32.1 (COL)
- net Col3: now also MX11.1 (COL), MX20.1 (COL), MX3.1 (COL), MX31.1 (COL), MX35.1 (COL), MX37.1 (COL), MX44.1 (COL), MX86.1 (COL), U1.14 (PB6); no longer MX1.1 (COL), MX102.1 (COL), MX21.1 (COL), MX23.1 (COL), MX24.1 (COL), MX25.1 (COL), MX29.1 (COL), MX6.1 (COL)
- net Col4: now also MX55.1 (COL), MX78.1 (COL), U1.15 (PB7); no longer MX47.1 (COL)
- net Col5: now also MX47.1 (COL), MX70.1 (COL), U1.16 (PB8); no longer MX55.1 (COL), MX78.1 (COL)
- net Col6: now also MX32.1 (COL), MX62.1 (COL), U1.17 (PB9); no longer MX39.1 (COL), MX70.1 (COL)
- net Col7: now also MX39.1 (COL), U1.18 (5V)
- net Col8: now also U1.19 (GND)
- net Col9: now also U1.20 (3V3)
- net GND: now also J1.4 (GND), U1.39 (GND)
- net Row1: now also U1.29 (PA3)
- net Row2: now also U1.30 (PA4)
- net Row3: now also U1.31 (PA5)
- net Row4: now also U1.32 (PA6)
- net Row5: now also U1.33 (PA7)
- net Row6: now also U1.34 (PB0)
- net Row7: now also U1.11 (PB3)
- net Row8: now also U1.10 (PA15)
- new net: D96.1 (K), R1.1
- new net: D104.1 (K), R2.1
- new net: D105.1 (K), R3.1
- new net +3V3: D104.2 (A), D105.2 (A), D96.2 (A), U1.38 (3V3)
- new net CAPS_LOCK: R2.2, U1.36 (PB2)
- new net D+: J1.3 (D+), U1.9 (PA12)
- new net D-: J1.2 (D-), U1.8 (PA11)
- new net NUM_LOCK: R1.2, U1.37 (PB10)
- new net SCROLL_LOCK: R3.2, U1.35 (PB1)
Other:
- moved on the sheet: D32, D39, D47, D55, D62, D70, D78, MX32, MX39, MX47, MX55, MX62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

Commit message: Created lib for logo
Parts:
- U1: symbol YAAJ_WeAct_BlackPill_Part_Like_SWD_Breakout:YAAJ_WeAct_BlackPill_Part_Like_SWD_Breakout -> ntc-6251-qmk-pcb-rescue:YAAJ_WeAct_BlackPill_Part_Like_SWD_Breakout-YAAJ_WeAct_BlackPill_Part_Like_SWD_Breakout
Changed lines of the file:
@@
 $EndComp
 $Comp
-L YAAJ_WeAct_BlackPill_Part_Like_SWD_Breakout:YAAJ_WeAct_BlackPill_Part_Like_SWD_Breakout U1
+L ntc-6251-qmk-pcb-rescue:YAAJ_WeAct_BlackPill_Part_Like_SWD_Breakout-YAAJ_WeAct_BlackPill_Part_Like_SWD_Breakout U1
 U 1 1 61C1A754
 P 7550 9000

Commit message: Changed connector fixed controller pins, re-routed all traces near controller
Parts:
- removed J1: USB_B, Connector_USB:USB_B_OST_USB-B1HSxx_Horizontal, symbol Connector:USB_B
- added J1: Conn_01x04_Male, Connector_PinHeader_2.54mm:PinHeader_1x04_P2.54mm_Horizontal, symbol Connector:Conn_01x04_Male
Connections:
- net +5V: now also J1.4 (Pin_4)
- net Col10: now also U1.24 (PC15); no longer U1.21 (VBat)
- net Col11: now also U1.25 (RES); no longer U1.22 (PC13)
- net Col12: now also U1.26 (PA0); no longer U1.23 (PC14)
- net Col13: now also U1.27 (PA1); no longer U1.24 (PC15)
- net Col7: now also U1.21 (VBat); no longer U1.18 (5V)
- net Col8: now also U1.22 (PC13); no longer U1.19 (GND)
- net Col9: now also U1.23 (PC14); no longer U1.20 (3V3)
- net D+: now also J1.2 (Pin_2)
- net D-: now also J1.3 (Pin_3)
- net GND: now also J1.1 (Pin_1)
Changed lines of the file:
@@
 Text GLabel 6650 9700 0    50   Input ~ 0
 Col6
-Text GLabel 6650 9800 0    50   Input ~ 0
+Text GLabel 8450 10000 2    50   Input ~ 0
 Col7
-Text GLabel 6650 9900 0    50   Input ~ 0
+Text GLabel 8450 9900 2    50   Input ~ 0
 Col8
-Text GLabel 6650 10000 0    50   Input ~ 0
+Text GLabel 8450 9800 2    50   Input ~ 0
 Col9
-Text GLabel 8450 10000 2    50   Input ~ 0
+Text GLabel 8450 9700 2    50   Input ~ 0
 Col10
-Text GLabel 8450 9900 2    50   Input ~ 0
+Text GLabel 8450 9600 2    50   Input ~ 0
 Col11
-Text GLabel 8450 9800 2    50   Input ~ 0
+Text GLabel 8450 9500 2    50   Input ~ 0
 Col12
-Text GLabel 8450 9700 2    50   Input ~ 0
+Text GLabel 8450 9400 2    50   Input ~ 0
 Col13
 Wire Wire Line
@@
 $EndComp
 $Comp
-L Connector:USB_B J1
-U 1 1 61E577A0
-P 12150 4850
-F 0 "J1" H 12207 5317 50  0000 C CNN
-F 1 "USB_B" H 12207 5226 50  0000 C CNN
-F 2 "Connector_USB:USB_B_OST_USB-B1HSxx_Horizontal" H 12300 4800 50  0001 C CNN
-F 3 " ~" H 12300 4800 50  0001 C CNN
-	1    12150 4850
-	1    0    0    -1
-$EndComp
-$Comp
 L ntc-6251-qmk-pcb-rescue:YAAJ_WeAct_BlackPill_Part_Like_SWD_Breakout-YAAJ_WeAct_BlackPill_Part_Like_SWD_Breakout U1
 U 1 1 61C1A754
@@
 L power:GND #PWR0101
 U 1 1 61C3454D
-P 12150 5250
-F 0 "#PWR0101" H 12150 5000 50  0001 C CNN
-F 1 "GND" H 12155 5077 50  0000 C CNN
-F 2 "" H 12150 5250 50  0001 C CNN
-F 3 "" H 12150 5250 50  0001 C CNN
-	1    12150 5250
-	1    0    0    -1
+P 12050 4800
+F 0 "#PWR0101" H 12050 4550 50  0001 C CNN
+F 1 "GND" H 12055 4627 50  0000 C CNN
+F 2 "" H 12050 4800 50  0001 C CNN
+F 3 "" H 12050 4800 50  0001 C CNN
+	1    12050 4800
+	0    -1   -1   0
 $EndComp
 $Comp
@@
 	0    1    1    0
 $EndComp
-Text GLabel 12450 4850 2    50   Input ~ 0
+Text GLabel 12050 4900 2    50   Input ~ 0
 D+
-Text GLabel 12450 4950 2    50   Input ~ 0
+Text GLabel 12050 5000 2    50   Input ~ 0
 D-
 Text GLabel 6650 8800 0    50   Input ~ 0
@@
 L power:+5V #PWR0104
 U 1 1 61C4D745
-P 12450 4650
-F 0 "#PWR0104" H 12450 4500 50  0001 C CNN
-F 1 "+5V" V 12465 4778 50  0000 L CNN
-F 2 "" H 12450 4650 50  0001 C CNN
-F 3 "" H 12450 4650 50  0001 C CNN
-	1    12450 4650
+P 12050 5100
+F 0 "#PWR0104" H 12050 4950 50  0001 C CNN
+F 1 "+5V" V 12065 5228 50  0000 L CNN
+F 2 "" H 12050 5100 50  0001 C CNN
+F 3 "" H 12050 5100 50  0001 C CNN
+	1    12050 5100
 	0    1    1    0
 $EndComp
@@
 Wire Wire Line
 	7350 6300 7350 6950
+$Comp
+L Connector:Conn_01x04_Male J1
+U 1 1 61CBF66C
+P 11850 4900
+F 0 "J1" H 11958 5181 50  0000 C CNN
+F 1 "Conn_01x04_Male" H 11958 5090 50  0000 C CNN
+F 2 "Connector_PinHeader_2.54mm:PinHeader_1x04_P2.54mm_Horizontal" H 11850 4900 50  0001 C CNN
+F 3 "~" H 11850 4900 50  0001 C CNN
+	1    11850 4900
+	1    0    0    -1
+$EndComp
 $EndSCHEMATC
