File: ntc-6251-qmk-pcb-rounded.kicad_pcb (KiCad board)
At the start: 2 copper layers, 432 x 109.1 mm, 212 parts, among them J1 USB_B, U1 YAAJ_WeAct_BlackPill_Part_Lik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

Commit message: Small fixes to rounded pcb
Routing:
- net Row8: track 261.9 -> 262.5 mm

Commit message: Finished most of small issues with traces
Parts:
- added G***: HVAJ, keyboard_parts:vicky_logo, F.Cu at (332.4, 140.6)
Routing:
- net Row6: track 465.7 -> 480.2 mm
- net Row8: track 262.5 -> 274.8 mm
- net Col8: track 576.8 -> 567.2 mm
- net Net-(D99-Pad2): track 0.00 -> 7.03 mm
- net Row7: track 293.7 -> 288.1 mm
- net Col12: track 442.9 -> 447.7 mm
- net Row1: track 353.8 -> 349.3 mm
- net Col3: track 462.7 -> 458.8 mm
- net Col2: track 474.3 -> 470.4 mm
- net Col5: track 635.3 -> 631.5 mm
- net Col4: track 632.2 -> 628.6 mm
- net Col10: track 452.3 -> 455.0 mm
- net Col7: track 630.5 -> 628.1 mm
- net Col6: track 649.5 -> 651.8 mm
- net Row5: track 303.6 -> 305.1 mm
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- added copper zone on B.Cu, net GND
- added copper zone on F.Cu, net GND

Commit message: Last fixes and copper pour on rounded pcb
Parts:
- removed the G*** at (332.4, 140.6)
- added G***: HVAJ, ntc-pcb:vicky_logo, F.Cu at (318.3, 142.1)
- J1: value USB_B -> Conn_01x04_Male; footprint Connector_USB:USB_B_OST_USB-B1HSxx_Horizontal -> Connector_PinHeader_2.54mm:PinHeader_1x04_P2.54mm_Horizontal; moved to F.Cu
- moved J1 4.83 mm to (389.8, 58.4)
- moved U1 2.90 mm to (369.9, 114.1)
Connections:
- J1 pad 1: +5V -> GND
- J1 pad 2: D- -> D+
- J1 pad 3: D+ -> D-
- J1 pad 4: GND -> +5V
- U1 pad 18: Col7 -> Net-(U1-Pad18)
- U1 pad 19: Col8 -> Net-(U1-Pad19)
- U1 pad 20: Col9 -> Net-(U1-Pad20)
- U1 pad 21: Col10 -> Col7
- U1 pad 22: Col11 -> Col8
- U1 pad 23: Col12 -> Col9
- U1 pad 24: Col13 -> Col10
- U1 pad 25: Net-(U1-Pad25) -> Col11
- U1 pad 26: Net-(U1-Pad26) -> Col12
- U1 pad 27: Net-(U1-Pad27) -> Col13
Routing:
- net Row7: track 288.1 -> 408.8 mm
- net Col6: track 651.8 -> 586.4 mm, vias 1 -> 2
- net Col7: track 628.1 -> 567.3 mm
- net Col12: track 447.7 -> 506.2 mm, vias 1 -> 0
- net Col8: track 567.2 -> 620.6 mm, vias 3 -> 2
- net Col5: track 631.5 -> 587.4 mm, vias 1 -> 2
- net Col4: track 628.6 -> 594.3 mm, vias 1 -> 2
- net Row8: track 274.8 -> 299.1 mm
- net Col9: track 411.9 -> 433.4 mm
- net GND: track 100.4 -> 83.6 mm, vias 8 -> 0
- net Row1: track 349.3 -> 362.7 mm
- net Net-(J1-Pad5): track 12.0 -> 0.00 mm
- net Col1: track 521.2 -> 509.2 mm
- net Col10: track 455.0 -> 443.3 mm
- net Row2: track 324.1 -> 334.4 mm
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- added copper zone on B.Cu, net (none)
- added copper zone on F.Cu, net (none)
- removed copper zone on B.Cu, net GND
- removed copper zone on F.Cu, net GND
