File: ntc-6251-qmk-pcb-rounded.kicad_pcb (KiCad board)
At the start: 2 copper layers, 432 x 109.1 mm, 213 parts, among them J1 Conn_01x04_Male, U1 YAAJ_WeAct_BlackPill_Part_Lik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

Commit message: Last small fixes before printing
Parts:
- moved G*** 61.0 mm to (379.3, 140.8)
Routing:
- net Col8: track 620.6 -> 631.7 mm
- net Col7: track 567.3 -> 578.1 mm
- net Row3: track 318.5 -> 323.6 mm
- net Row6: track 477.8 -> 475.0 mm
- net Row2: track 334.4 -> 335.4 mm
- net Col12: track 506.2 -> 505.4 mm

Commit message: Output file added to project
Other:
- board text added: "JLCJLCJLCJLC"
Changed lines of the file:
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@@
   (general
     (thickness 1.6)
-    (drawings 126)
+    (drawings 127)
     (tracks 5356)
     (zones 0)
@@
       (outputformat 1)
       (mirror false)
-      (drillshape 1)
+      (drillshape 0)
       (scaleselection 1)
-      (outputdirectory ""))
+      (outputdirectory "output"))
   )
   (net 0 "")
@@
     )
   )
+  (gr_text JLCJLCJLCJLC (at 215.86 154.88) (layer F.SilkS)
+    (effects (font (size 1.5 1.5) (thickness 0.3)))
+  )
   (gr_line (start 320.25214 134.28) (end 344.85214 134.28) (layer Dwgs.User) (width 0.15))
