File: pcb/ntc-6251-qmk-pcb.kicad_pcb (KiCad board)
At the start: 2 copper layers, 432 x 109.1 mm, 213 parts, among them J1 Conn_01x04_Male, U1 YAAJ_WeAct_BlackPill_Part_Lik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

Commit message: Added via layout json and found some bugs
Connections:
- U1 pad 21: Col7 -> Net-(U1-Pad21)
- U1 pad 25: Col11 -> Net-(U1-Pad25)
- U1 pad 28: Net-(U1-Pad28) -> Col11
- U1 pad 7: Net-(U1-Pad7) -> Col7
