File: pcb/ntc-6251-qmk-pcb.sch (KiCad schematic (older format))
At the start: 212 parts, among them J1 Conn_01x04_Male, U1 YAAJ_WeAct_BlackPill_Part_Lik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

Commit message: Cleanup
Parts:
- U1: symbol ntc-6251-qmk-pcb-rescue:YAAJ_WeAct_BlackPill_Part_Like_SWD_Breakout-YAAJ_WeAct_BlackPill_Part_Like_SWD_Breakout -> YAAJ_WeAct_BlackPill_Part_Like_SWD_Breakout:YAAJ_WeAct_BlackPill_Part_Like_SWD_Breakout
Changed lines of the file:
@@
 $EndComp
 $Comp
-L ntc-6251-qmk-pcb-rescue:YAAJ_WeAct_BlackPill_Part_Like_SWD_Breakout-YAAJ_WeAct_BlackPill_Part_Like_SWD_Breakout U1
+L YAAJ_WeAct_BlackPill_Part_Like_SWD_Breakout:YAAJ_WeAct_BlackPill_Part_Like_SWD_Breakout U1
 U 1 1 61C1A754
 P 7550 9000

Commit message: Switched place for schematic column 1 and 3
Other:
- moved on the sheet: D1, D102, D11, D20, D21, D23, D24, D25, D29, D3, D31, D35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

Commit message: Added via layout json and found some bugs
Connections:
- net Col11: now also U1.28 (PA2); no longer U1.25 (RES)
- net Col7: now also U1.7 (PA10); no longer U1.21 (VBat)
Other:
- note added: "Col7 was placed on VBat\nCol11 was placed on RES"
- note added: "Consider moving Col8 from C13 since the led blinks when active"
Changed lines of the file:
@@
 Text GLabel 6650 9700 0    50   Input ~ 0
 Col6
-Text GLabel 8450 10000 2    50   Input ~ 0
+Text GLabel 6650 8700 0    50   Input ~ 0
 Col7
 Text GLabel 8450 9900 2    50   Input ~ 0
@@
 Text GLabel 8450 9700 2    50   Input ~ 0
 Col10
-Text GLabel 8450 9600 2    50   Input ~ 0
+Text GLabel 8450 9300 2    50   Input ~ 0
 Col11
 Text GLabel 8450 9500 2    50   Input ~ 0
@@
 Connection ~ 5250 3450
 Connection ~ 5250 2800
+Text Notes 8150 10350 0    50   ~ 0
+Col7 was placed on VBat\nCol11 was placed on RES
+Text Notes 8150 10450 0    50   ~ 0
+Consider moving Col8 from C13 since the led blinks when active
 $EndSCHEMATC

Commit message: Further notes added to schematic about A0 being connected to user button
Connections:
- no-connect marks 0 -> 11
Other:
- note added: "A0 is connected to the user button, pressing it connects the whole column/row to gnd, effectively pressing all buttons..."
Changed lines of the file:
@@
 Connection ~ 5250 3450
 Connection ~ 5250 2800
-Text Notes 8150 10350 0    50   ~ 0
+Text Notes 5800 10500 0    50   ~ 0
 Col7 was placed on VBat\nCol11 was placed on RES
-Text Notes 8150 10450 0    50   ~ 0
+Text Notes 5800 10600 0    50   ~ 0
 Consider moving Col8 from C13 since the led blinks when active
+Text Notes 5800 10700 0    50   ~ 0
+A0 is connected to the user button, pressing it connects the whole column/row to gnd, effectively pressing all buttons...
+NoConn ~ 8450 10000
+NoConn ~ 8450 9600
+NoConn ~ 6650 10000
+NoConn ~ 6650 9900
+NoConn ~ 6650 9800
+NoConn ~ 6650 8600
+NoConn ~ 6650 8500
+NoConn ~ 6650 8400
+NoConn ~ 6650 8300
+NoConn ~ 6650 8200
+NoConn ~ 6650 8100
 $EndSCHEMATC

Commit message: Futher notes
Other:
- note added: "A0 is connected to the user button, pressing it connects the whole column/row to gnd, effectively pressing all buttons...\n"
- note added: "Col7 was placed on VBat\nCol11 was placed on RES and A2 was unoccupied"
- note added: "Consider moving Col8 from C13 since the led blinks when active. Tested with alps switch and doesn't affect function"
- note removed: "A0 is connected to the user button, pressing it connects the whole column/row to gnd, effectively pressing all buttons..."
- note removed: "Col7 was placed on VBat\nCol11 was placed on RES"
- note removed: "Consider moving Col8 from C13 since the led blinks when active"
Changed lines of the file:
@@
 Connection ~ 5250 2800
 Text Notes 5800 10500 0    50   ~ 0
-Col7 was placed on VBat\nCol11 was placed on RES
+Col7 was placed on VBat\nCol11 was placed on RES and A2 was unoccupied
 Text Notes 5800 10600 0    50   ~ 0
-Consider moving Col8 from C13 since the led blinks when active
+Consider moving Col8 from C13 since the led blinks when active. Tested with alps switch and doesn't affect function
 Text Notes 5800 10700 0    50   ~ 0
-A0 is connected to the user button, pressing it connects the whole column/row to gnd, effectively pressing all buttons...
+A0 is connected to the user button, pressing it connects the whole column/row to gnd, effectively pressing all buttons...\n
 NoConn ~ 8450 10000
 NoConn ~ 8450 9600
